File: rgb-board.kicad_sch (KiCad schematic)
At the start: 84 parts, among them J1 Conn_02x25_Odd_Even, J2 SCART-F, J5 DE15_Plug_HighDensity_Mountin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, J6 SJ1-3535NG, K1 G6K-2PY-12DC, Q101 BC850C, Q105 BC850C, Q109 BC850C, Q113 BC850C, Q114 BC850C, Q201 BC850C, SW1 SW_DPDT_x2, SW2 SPUJ193700, U1 NCP1117-12_SOT223

Commit message: SCART / VGA switching schematic.
Connections:
- net +12V: now also SW2.3 (B1)
- net B/B-Y: no longer J2.7 (P7)
- net G/Y: no longer J2.11 (P11)
- net GND: now also K1.8
- net HD/CS: no longer J2.20 (P20)
- net H_SYNC: now also K1.4
- net R/R-Y: no longer J2.15 (P15)
- net VD: now also K1.6
- net VGA_B: now also SW2.6 (B2)
- net VGA_G: now also SW2.9 (B3)
- net VGA_R: now also SW2.12 (B4)
- net V_SYNC: now also K1.5
- net VGA_SELECT: now reaches K1.1
- net VGA_SELECT: now also SW2.2 (COM1)
- net SCART_SYNC: now reaches K1.2
- net SCART_SYNC: now also J2.20 (P20)
- net HD/CS: now reaches K1.3
- net SCART_R: now reaches SW2.10 (A4)
- net SCART_R: now also J2.15 (P15)
- net R/R-Y: now reaches SW2.11 (COM4)
- net SCART_B: now reaches SW2.4 (A2)
- net SCART_B: now also J2.7 (P7)
- net B/B-Y: now reaches SW2.5 (COM2)
- net SCART_G: now reaches SW2.7 (A3)
- net SCART_G: now also J2.11 (P11)
- net G/Y: now reaches SW2.8 (COM3)
- no-connect marks 42 -> 44
Other:
- moved on the sheet: K1, SW2
