File: rgb-board.kicad_sch (KiCad schematic)
At the start: 84 parts, among them J1 Conn_02x25_Odd_Even, J2 SCART-F, J5 DE15_Plug_HighDensity_Mountin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, J6 SJ1-3535NG, K1 G6K-2PY-12DC, Q101 BC850C, Q105 BC850C, Q109 BC850C, Q113 BC850C, Q114 BC850C, Q201 BC850C, SW1 SW_DPDT_x2, SW2 SPUJ193700, U1 NCP1117-12_SOT223

Commit message: Add ALPS SPUJ Series push switches footprints library. Replace LC2259 and PBH4UEE push switches with ALPS SPUJ190900 and SPUJ193700. Remove LC2259 and PBH4UEE footprints.
Parts:
- SW1: footprint LC2259:LC2259 -> ALPS_SPUJ:SPUJ190900
- SW2: footprint PBH4UEE:PBH4UEE -> ALPS_SPUJ:SPUJ193700
Changed lines of the file:
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@@
 			)
 		)
-		(property "Footprint" "LC2259:LC2259"
+		(property "Footprint" "ALPS_SPUJ:SPUJ190900"
 			(at 91.44 154.94 0)
 			(effects
@@
 			)
 		)
-		(property "Footprint" "LC2259:LC2259"
+		(property "Footprint" "ALPS_SPUJ:SPUJ190900"
 			(at 91.44 170.18 0)
 			(effects
@@
 			)
 		)
-		(property "Footprint" "PBH4UEE:PBH4UEE"
+		(property "Footprint" "ALPS_SPUJ:SPUJ193700"
 			(at 95.25 240.03 0)
 			(effects

Commit message: Route PCB.
+14V power line polyfuse added.
Parts:
- added F1: 1812L050PR, Fuse:Fuse_1812_4532Metric_Pad1.30x3.40mm_HandSolder, symbol Device:Polyfuse
Connections:
- net AUDIO_EXT_L: now also SW1.3 (C); no longer SW1.6 (C)
- net AUDIO_EXT_R: now also SW1.6 (C); no longer SW1.3 (C)
- net AUDIO_INT_L: now also SW1.1 (A); no longer SW1.4 (A)
- net AUDIO_INT_R: now also SW1.4 (A); no longer SW1.1 (A)
- net AUDIO_L: now also SW1.2 (B); no longer SW1.5 (B)
- net AUDIO_R: now also SW1.5 (B); no longer SW1.2 (B)
- net G/Y: now also SW2.11 (COM4); no longer SW2.8 (COM3)
- net HD/CS: now also K1.6; no longer K1.3
- net H_SYNC: now also K1.5; no longer K1.4
- net R/R-Y: now also SW2.8 (COM3); no longer SW2.11 (COM4)
- net SCART_G: now also SW2.10 (A4); no longer SW2.7 (A3)
- net SCART_R: now also SW2.7 (A3); no longer SW2.10 (A4)
- net SCART_SYNC: now also K1.7; no longer K1.2
- net VCC+14V: now also F1.1; no longer C122.1, U1.3 (VI)
- net VD: now also K1.3; no longer K1.6
- net VGA_G: now also SW2.12 (B4); no longer SW2.9 (B3)
- net VGA_R: now also SW2.9 (B3); no longer SW2.12 (B4)
- net V_SYNC: now also K1.4; no longer K1.5
- new net: C122.1, F1.2, U1.3 (VI)
- no-connect marks 44 -> 45
Other:
- moved on the sheet: J5, J6, K1, SW2

Commit message: Correct R203, R205 resistors marking for BoM.
Parts:
- R203: value 56K -> 56k
- R205: value 2.7K -> 2.7k
Changed lines of the file:
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@@
 			)
 		)
-		(property "Value" "56K"
+		(property "Value" "56k"
 			(at 146.05 110.49 90)
 			(effects
@@
 			)
 		)
-		(property "Value" "2.7K"
+		(property "Value" "2.7k"
 			(at 161.29 128.27 90)
 			(effects

Commit message: Fixed Relay_DPDT_Omron_G6K-2P footprint pins spacing according to datasheet. Footprint copied from KiCad 8.0.0 global library to project.
Fixed BOM duplicated values.
Parts:
- K1: footprint Relay_THT:Relay_DPDT_Omron_G6K-2P -> Omron_G6K-2P:Relay_DPDT_Omron_G6K-2P
Changed lines of the file:
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@@
 			)
 		)
-		(property "Footprint" "Relay_THT:Relay_DPDT_Omron_G6K-2P"
+		(property "Footprint" "Omron_G6K-2P:Relay_DPDT_Omron_G6K-2P"
 			(at 140.97 219.71 0)
 			(effects
